File: design_files/AST1025.brd (EAGLE design)
At the start: 10 x 10 mm, 7 parts, among them J1 SM05B, U2 BME280

Commit message: updates
Parts:
- C1: value 10uF -> 1uF
- J1: device tinycircuits:JST_SH_5X1 -> tinycircuits:JST_SH_5X1_EDGE
Other:
- board text added: "Humidity"
- board text added: "Pressure"
- board text added: "R2"
- board text added: "Wireling Pressure Humidity"
- board text removed: "Pres/Hum"
- board text removed: "Pressure & Humidity Sensor"
- board text removed: "Sensor R2"
Changed lines of the file:
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@@
 <layer number="59" name="Invisible" color="7" fill="1" visible="no" active="no"/>
 <layer number="61" name="stand" color="7" fill="1" visible="no" active="no"/>
+<layer number="88" name="SimResults" color="9" fill="1" visible="yes" active="yes"/>
+<layer number="89" name="SimProbes" color="9" fill="1" visible="yes" active="yes"/>
 <layer number="90" name="Modules" color="5" fill="1" visible="yes" active="yes"/>
 <layer number="91" name="Nets" color="2" fill="1" visible="no" active="no"/>
@@
 <layer number="158" name="bResistor" color="7" fill="1" visible="no" active="yes"/>
 <layer number="159" name="henwayCAP" color="13" fill="1" visible="yes" active="yes"/>
+<layer number="160" name="IDFDebug" color="7" fill="1" visible="yes" active="yes"/>
 <layer number="191" name="mNets" color="7" fill="1" visible="no" active="no"/>
 <layer number="192" name="mBusses" color="7" fill="1" visible="no" active="no"/>
@@
 <wire x1="0" y1="40.8" x2="0" y2="0" width="0.127" layer="48"/>
 <dimension x1="15" y1="20" x2="25" y2="20" x3="20" y3="21.454653125" layer="48"/>
-<text x="38.111025" y="4.365003125" size="0.889" layer="48">Pressure &amp; Humidity Sensor</text>
+<text x="38.111025" y="4.365003125" size="0.889" layer="48">Wireling Pressure Humidity</text>
 <text x="34.986825" y="1.7714" size="0.889" layer="48">AS-PCB-AST1025</text>
 <text x="57.3810375" y="1.6952" size="0.889" layer="48">2</text>
@@
 <rectangle x1="18.747940625" y1="13.71801875" x2="19.027340625" y2="13.72309375" layer="22"/>
 <rectangle x1="20.8155" y1="13.71801875" x2="21.08981875" y2="13.72309375" layer="22"/>
-<text x="21.5" y="16.4" size="0.76" layer="22" rot="SMR0">Pres/Hum</text>
+<text x="21.5" y="16.4" size="0.76" layer="22" rot="SMR0">Pressure</text>
 <wire x1="22" y1="14.45" x2="23.15" y2="15.65" width="0.1" layer="22"/>
 <wire x1="22" y1="15.05" x2="22.55" y2="15.6" width="0.1" layer="22"/>
@@
 <wire x1="22" y1="15.75" x2="22" y2="15.05" width="0.1" layer="22"/>
 <wire x1="22" y1="15.05" x2="22" y2="14.45" width="0.1" layer="22"/>
-<text x="21.5" y="15.4" size="0.762" layer="22" rot="SMR0">Sensor R2</text>
+<text x="21.5" y="15.4" size="0.762" layer="22" rot="SMR0">Humidity</text>
 <hole x="16.5" y="18.5" drill="1.5"/>
 <hole x="23.5" y="18.5" drill="1.5"/>
 <text x="21.5" y="14.4" size="0.762" layer="22" rot="SMR0">AST1025</text>
+<text x="21.5" y="17.5" size="0.76" layer="22" rot="SMR0">R2</text>
 </plain>
 <attributes>
@@
 <attribute name="VALUE" value="0.1uF" x="19.65" y="19.45" size="1.778" layer="27" display="off"/>
 </element>
-<element name="C1" library="tinycircuits" package="C0603" value="10uF" x="24.2" y="14.2" rot="R90">
-<attribute name="PARTNO" value="AS-ITM-00002" x="24.2" y="14.2" size="1.778" layer="27" rot="R90" display="off"/>
-<attribute name="VALUE" value="10uF" x="24.2" y="14.2" size="1.778" layer="27" rot="R90" display="off"/>
+<element name="C1" library="tinycircuits" package="C0603" value="1uF" x="24.2" y="14.2" rot="R90">
+<attribute name="PARTNO" value="AS-ITM-00410" x="24.2" y="14.2" size="1.778" layer="27" rot="R90" display="off"/>
+<attribute name="VALUE" value="1uF" x="24.2" y="14.2" size="1.778" layer="27" rot="R90" display="off"/>
 </element>
-<element name="J1" library="tinycircuits" package="JST_SH_5X1" value="SM05B" x="20" y="12.125">
+<element name="J1" library="tinycircuits" package="JST_SH_5X1_EDGE" value="SM05B" x="20" y="12.125">
 <attribute name="PARTNO" value="AS-ITM-00340" x="20" y="12.125" size="1.778" layer="27" display="off"/>
 <attribute name="VALUE" value="SM05B" x="20" y="12.125" size="1.778" layer="27" display="off"/>
