File: design_files/AST1025.sch (EAGLE design)
At the start: 6 parts, among them J1 SM05B, U2 BME280

Commit message: updates
Parts:
- C1: value 10uF -> 1uF; device tinycircuits:AS-ITM-00002 -> tinycircuits:AS-ITM-00410; PARTNO (none) -> AS-ITM-00410; VALUE (none) -> 1uF
- J1: device tinycircuits:AS-ITM-00340 -> tinycircuits:AS-ITM-00340EDGE
Other:
- note added: "Non Populated: R2"
- note added: "Variant: Standard - R"
- note added: "Wireling Pressure Humidity"
- note removed: "NOTES:"
- note removed: "NP: R1"
- note removed: "Non Populated: R1"
- note removed: "Pressure & Humidity Sensor"
- note removed: "Variant: Standard"
